File: buck.brd (EAGLE design)
At the start: 100 x 100 mm, 32 parts, among them J1 B06B-HCMKK, J2 POWERPOLE_POWER45A_DRILL, J3 POWERPOLE_POWER45A_DRILL

Commit message: Add files via upload
Parts:
- renumbered U$4 to CHOKEME
Other:
- board text added: "1.6abuck"
- board text added: "150uH"
- board text added: "6abuck"
- board text added: "Samthemam"
- board text added: "bruh"
- board text added: "yousofine"
- board text added: "yugbug"
Changed lines of the file:
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@@
 <wire x1="100" y1="100" x2="0" y2="100" width="0" layer="20"/>
 <wire x1="0" y1="100" x2="0" y2="0" width="0" layer="20"/>
+<text x="9" y="28" size="1.778" layer="25">yugbug</text>
+<text x="26" y="44" size="1.778" layer="25">150uH</text>
+<text x="39" y="3" size="1.778" layer="25">Samthemam</text>
+<text x="66" y="12" size="1.778" layer="25">yousofine</text>
+<text x="2" y="2" size="1.778" layer="25">bruh</text>
+<text x="67" y="27" size="1.778" layer="25">1.6abuck</text>
+<text x="62" y="68" size="1.778" layer="25">6abuck</text>
 </plain>
 <attributes>
@@
 </variantdefs>
 <classes>
-<class number="0" name="default" width="0.381" drill="0">
+<class number="0" name="default" width="0.762" drill="0">
 </class>
 <class number="1" name="Power" width="1.524" drill="0">
@@
 <autorouter>
 <pass name="Default">
-<param name="RoutingGrid" value="0.125mm"/>
+<param name="RoutingGrid" value="4.92125984mil"/>
 <param name="AutoGrid" value="1"/>
 <param name="Efforts" value="2"/>
@@
 <element name="U$2" library="REV BLDC" package="MINI-SB-50" value="SB50" x="9.58" y="81.78" smashed="yes"/>
 <element name="U$3" library="buck_1.6" package="BUCK1.6A" value="BUCK1.6A" x="71.36" y="31.37" smashed="yes"/>
-<element name="U$4" library="cmnModeChoke1.2mH" package="CMNMODECHOKE1.2MH" value="CMNMODECHOKE1.2MH" x="27.8" y="15.32" smashed="yes"/>
+<element name="CHOKEME" library="cmnModeChoke1.2mH" package="CMNMODECHOKE1.2MH" value="CMNMODECHOKE1.2MH" x="27.8" y="15.32" smashed="yes"/>
 </elements>
 <signals>
@@
 <contactref element="BUCK150UH" pad="2"/>
 <contactref element="TP12" pad="TP"/>
-<contactref element="U$4" pad="1"/>
+<contactref element="CHOKEME" pad="1"/>
 <contactref element="C3" pad="1"/>
 <wire x1="34" y1="29.5" x2="35" y2="29.5" width="0.381" layer="1"/>
@@
 <signal name="N$4">
 <contactref element="C3" pad="2"/>
-<contactref element="U$4" pad="4"/>
+<contactref element="CHOKEME" pad="4"/>
 <contactref element="BUCK150UH" pad="3"/>
 <contactref element="TP13" pad="TP"/>
@@
 <wire x1="40.5" y1="47" x2="40.512" y2="47.32" width="0.381" layer="1"/>
 <wire x1="39.5" y1="29.5" x2="39.15" y2="29.3" width="0.381" layer="1"/>
-<wire x1="40.5" y1="47.5" x2="40.5" y2="53" width="0.381" layer="1"/>
-<wire x1="40.5" y1="53" x2="40.18" y2="53.03" width="0.381" layer="1"/>
+<wire x1="40.5" y1="47.5" x2="40.5" y2="53" width="0.762" layer="1"/>
+<wire x1="40.5" y1="53" x2="40.18" y2="53.03" width="0.762" layer="1"/>
 <wire x1="40.5" y1="47.5" x2="40.512" y2="47.32" width="0.381" layer="1"/>
 </signal>
@@
 </signal>
 <signal name="N$6">
-<contactref element="U$4" pad="2"/>
+<contactref element="CHOKEME" pad="2"/>
 <contactref element="U$3" pad="+VIN"/>
 <contactref element="TP9" pad="TP"/>
@@
 <contactref element="C5" pad="1"/>
 <contactref element="U$3" pad="-VIN"/>
-<contactref element="U$4" pad="3"/>
+<contactref element="CHOKEME" pad="3"/>
 <contactref element="TP10" pad="TP"/>
 <wire x1="83.5" y1="56.5" x2="83.5" y2="68" width="0.381" layer="1"/>

Commit message: Add files via upload
Fattened some of the traces
Parts:
- moved TP7 8.60 mm to (55.1, 71.4)
- moved TP6 2.00 mm to (49.2, 91.4)
- moved J2 1.41 mm to (92.5, 23.2)
Routing:
- net 1.6A_OUT: track 153.0 -> 158.8 mm
- net RC: track 37.8 -> 42.1 mm
- net 6A_OUT: track 109.6 -> 110.7 mm
- net N$6: track 68.0 -> 68.6 mm
Other:
- board text removed: "Samthemam"
- board text removed: "bruh"
- board text removed: "yousofine"
- board text removed: "yugbug"
