File: buck.sch (EAGLE design)
At the start: 32 parts, among them J1 B06B-HCMKK, J2 POWERPOLE_POWER45A_DRILL, J3 POWERPOLE_POWER45A_DRILL

Commit message: Add files via upload
Parts:
- renumbered U$4 to CHOKEME
Changed lines of the file:
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@@
 </variantdefs>
 <classes>
-<class number="0" name="default" width="0.381" drill="0">
+<class number="0" name="default" width="0.762" drill="0">
 </class>
 <class number="1" name="Power" width="1.524" drill="0">
@@
 <part name="C1" library="rcl" library_urn="urn:adsk.eagle:library:334" deviceset="EL-" device="BI25-10AXIAL" package3d_urn="urn:adsk.eagle:package:23718/1" value="10uF"/>
 <part name="R2" library="rcl" library_urn="urn:adsk.eagle:library:334" deviceset="R-US_" device="R0805" package3d_urn="urn:adsk.eagle:package:23553/2" value="100 ohm"/>
-<part name="U$4" library="cmnModeChoke1.2mH" deviceset="CMNMODECHOKE1.2MH" device=""/>
+<part name="CHOKEME" library="cmnModeChoke1.2mH" deviceset="CMNMODECHOKE1.2MH" device=""/>
 <part name="R1" library="rcl" library_urn="urn:adsk.eagle:library:334" deviceset="R-US_" device="R0805" package3d_urn="urn:adsk.eagle:package:23553/2" value="390 ohm"/>
 <part name="LED2" library="led" library_urn="urn:adsk.eagle:library:259" deviceset="LED" device="CHIP-LED0603" package3d_urn="urn:adsk.eagle:package:15819/3"/>
@@
 <attribute name="VALUE" x="69.85" y="42.418" size="1.778" layer="96"/>
 </instance>
-<instance part="U$4" gate="G$1" x="-2.54" y="-20.32" smashed="yes"/>
+<instance part="CHOKEME" gate="G$1" x="-2.54" y="-20.32" smashed="yes"/>
 <instance part="R1" gate="G$1" x="83.82" y="27.94" smashed="yes">
 <attribute name="NAME" x="80.01" y="29.4386" size="1.778" layer="95"/>
@@
 <wire x1="-33.34" y1="-13.78" x2="-33.34" y2="-15.24" width="0.1524" layer="91"/>
 <wire x1="-33.34" y1="-15.24" x2="-22.86" y2="-15.24" width="0.1524" layer="91"/>
-<pinref part="U$4" gate="G$1" pin="1"/>
+<pinref part="CHOKEME" gate="G$1" pin="1"/>
 <wire x1="-12.7" y1="-15.24" x2="-22.86" y2="-15.24" width="0.1524" layer="91"/>
 <junction x="-22.86" y="-15.24"/>
@@
 <segment>
 <pinref part="C3" gate="G$1" pin="2"/>
-<pinref part="U$4" gate="G$1" pin="4"/>
+<pinref part="CHOKEME" gate="G$1" pin="4"/>
 <wire x1="-12.7" y1="-25.4" x2="-22.86" y2="-25.4" width="0.1524" layer="91"/>
 <junction x="-22.86" y="-25.4"/>
@@
 <net name="N$6" class="0">
 <segment>
-<pinref part="U$4" gate="G$1" pin="2"/>
+<pinref part="CHOKEME" gate="G$1" pin="2"/>
 <wire x1="7.62" y1="-15.24" x2="20.32" y2="-15.24" width="0.1524" layer="91"/>
 <pinref part="U$3" gate="G$1" pin="+VIN"/>
@@
 <wire x1="10.16" y1="-35.56" x2="15.24" y2="-35.56" width="0.1524" layer="91"/>
 <wire x1="24.8" y1="-21.4" x2="10.16" y2="-21.4" width="0.1524" layer="91"/>
-<pinref part="U$4" gate="G$1" pin="3"/>
+<pinref part="CHOKEME" gate="G$1" pin="3"/>
 <wire x1="10.16" y1="-21.4" x2="10.16" y2="-22.86" width="0.1524" layer="91"/>
 <wire x1="10.16" y1="-22.86" x2="10.16" y2="-25.4" width="0.1524" layer="91"/>
